File: anarchitechno-box/kicad/isolators.kicad_sch (KiCad schematic)
At the start: 10 parts, among them U13 ISO7740DWR, U14 ISO7740DWR, U15 ISO7742DWR

Commit message: meer Stijn in de Trein
Connections:
- net +3.3V renamed +3V3

Commit message: Resized PCB with mounts at 125x125mm (suitable for 140mm PC fan), 4-pin fan connector added, changed 3.3VP to 5.0VP
Connections:
- net +3.3VP renamed +5VP

Commit message: Schematic & PCB changes: - Cleaned up unnecessary electrolytic input capacitor flyback - Removed dual diode rectification on 5V, increased output capacitors - Feedback resistors DC/DCs set, enlarged for JLC basic parts - Sweep through schematic to consolidate caps to JLC basic parts (see list schematic front page) - Midi OUTPUT added (please check schematic) - Wiznet W5500 schematic reworked to RJ45 reference schematic: https://docs.wiznet.io/assets/files/w5500_sch_v110_use_mag_-dfff8bbb103d13be4f25cd2b2f8b950d.pdf - Replaced ethernet jack to HR911105A - Crystals chosen for W5500 and RP2350B (according to reference), 15pF load caps. - RS485 driver changed to SP3485EN for 3.3V operation - Replaced RS485 bus connectors with 2x RJ45s for passthrough - Groove connector replaced with JST XH 2mm - Added LCSC part numbers for various components in the schematic
Parts:
- U13, U14: LCSC Part (none) -> C529547
- U15: LCSC Part (none) -> C529288
Changed lines of the file:
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@@
+			)
+		)
+		(property "LCSC Part" "C529547"
+			(at 90.17 30.48 0)
+			(effects
+				(font
+					(size 1.27 1.27)
+				)
+				(hide yes)
 			)
 		)
@@
 			)
 		)
+		(property "LCSC Part" "C529288"
+			(at 90.17 125.73 0)
+			(effects
+				(font
+					(size 1.27 1.27)
+				)
+				(hide yes)
+			)
+		)
 		(pin "11"
 		)
@@
 			(effects
 				(font
+					(size 1.27 1.27)
+				)
+				(hide yes)
+			)
+		)
+		(property "LCSC Part" "C529547"
+			(at 90.17 77.47 0)
+			(effects
+				(font
