File: anarchitechno-box/kicad/TwoIsolatedFETs.kicad_sch (KiCad schematic)
At the start: 2 parts, among them U1 TC4426xOA, U2 ADuM1200AR

Commit message: Large intermediate schematic push. Remaining todos are on frontpage.
Parts:
- removed U1: TC4426xOA, Package_SO:SOIC-8_3.9x4.9mm_P1.27mm, symbol Driver_FET:TC4426xOA
- removed U2: ADuM1200AR, Package_SO:SOIC-8_3.9x4.9mm_P1.27mm, symbol Isolator:ADuM1200AR
- added C30, C31: 100nF, Capacitor_SMD:C_0402_1005Metric, symbol Device:C
- added D4: BAT54AW, Package_TO_SOT_SMD:SOT-323_SC-70, symbol Diode:BAT54AW
- added U9: ISO7740DWR, Package_SO:SOIC-16W_7.5x10.3mm_P1.27mm, symbol parts:ISO7740
Connections:
- net +3.3V: now also C30.1, U9.1 (VCC1)
- net GND: now also C30.2, U9.2 (GND1), U9.8 (GND1)
- net GND2: now also C31.2, U9.15 (GND2), U9.9 (GND2)
- new net +3.3VP: C31.1, U9.10 (EN2), U9.16 (VCC2)
- new net DRV_nFAULT_COMMON: D4.3
- new net HBridge_A/DRV_nFAULT: D4.1
- new net HBridge_A/PWM_1: U9.14 (OUTA)
- new net HBridge_A/PWM_2: U9.13 (OUTB)
- new net HBridge_B/DRV_nFAULT: D4.2
- new net HBridge_B/PWM_1: U9.12 (OUTC)
- new net HBridge_B/PWM_2: U9.11 (OUTD)
- new net MCU_PWM_A_1: U9.3 (INA)
- new net MCU_PWM_A_2: U9.4 (INB)
- new net MCU_PWM_B_1: U9.5 (INC)
- new net MCU_PWM_B_2: U9.6 (IND)
- no-connect marks 0 -> 3
Other:
- removed sheet FET
- removed sheet FET1
- added sheet HBridge_A (hbridge.kicad_sch)
- added sheet HBridge_B (hbridge.kicad_sch)

Commit message: meer Stijn in de Trein
Connections:
- net HBridge_A/DRV_nFAULT: now also D4.2; no longer D4.1
- net HBridge_B/DRV_nFAULT: now also D4.1; no longer D4.2
- net +3.3V renamed +3V3
- net HBridge_A/PWM_1 renamed PWM_A_2
- net HBridge_A/PWM_2 renamed PWM_A_1
- net HBridge_B/PWM_1 renamed PWM_B_2
- net HBridge_B/PWM_2 renamed PWM_B_1

Commit message: Resized PCB with mounts at 125x125mm (suitable for 140mm PC fan), 4-pin fan connector added, changed 3.3VP to 5.0VP
Connections:
- net +3.3VP renamed +5VP
Changed lines of the file:
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@@
+	)
+	(symbol
+		(lib_id "power:+5VP")
+		(at 114.3 85.09 0)
+		(unit 1)
+		(exclude_from_sim no)
+		(in_bom yes)
+		(on_board yes)
+		(dnp no)
+		(fields_autoplaced yes)
+		(property "Reference" "#PWR034"
+			(at 114.3 88.9 0)
+			(effects
+				(font
+					(size 1.27 1.27)
+				)
+				(hide yes)
+			)
+		)
+		(property "Value" "+5VP"
+			(at 114.3 80.01 0)
+			(effects
+				(font
+					(size 1.27 1.27)
+				)
+			)
+		)
+		(property "Footprint" ""
+			(at 114.3 85.09 0)
+			(effects
+				(font
+					(size 1.27 1.27)
+				)
+				(hide yes)
+			)
+		)
+		(property "Datasheet" ""
+			(at 114.3 85.09 0)
+			(effects
+				(font
+					(size 1.27 1.27)
+				)
+				(hide yes)
+			)
+		)
+		(property "Description" "Power symbol creates a global label with name \"+5VP\""
+			(at 114.3 85.09 0)
+			(effects
+				(font
+					(size 1.27 1.27)
+				)
+				(hide yes)
+			)
+		)
+		(pin "1"
+		)
+		(instances
+			(project "anarchytechnobox"
+				(path "/8c734c41-38ed-40fc-83bd-134786dcfb35/48f260d8-d62f-49a9-8985-05fca65ac6cb"
+					(reference "#PWR034")
+					(unit 1)
+				)
+				(path "/8c734c41-38ed-40fc-83bd-134786dcfb35/f97c65ed-bb3f-4eb8-a2c6-056cc510b5f8"
+					(reference "#PWR057")
+					(unit 1)
+				)
+			)
+		)
 	)
 	(symbol
@@
 	)
 	(symbol
-		(lib_id "power:+3.3VP")
-		(at 114.3 85.09 0)
-		(unit 1)
-		(exclude_from_sim no)
-		(in_bom yes)
-		(on_board yes)
-		(dnp no)
-		(fields_autoplaced yes)
-		(property "Reference" "#PWR057"
-			(at 118.11 86.36 0)
-			(effects
-				(font
-					(size 1.27 1.27)
-				)
-				(hide yes)
-			)
-		)
-		(property "Value" "+3.3VP"
-			(at 114.3 80.01 0)
-			(effects
-				(font
-					(size 1.27 1.27)
-				)
-			)
-		)
-		(property "Footprint" ""
-			(at 114.3 85.09 0)
-			(effects
-				(font
-					(size 1.27 1.27)
-				)
-				(hide yes)
-			)
-		)
-		(property "Datasheet" ""
-			(at 114.3 85.09 0)
-			(effects
-				(font
-					(size 1.27 1.27)
-				)
-				(hide yes)
-			)
-		)
-		(property "Description" "Power symbol creates a global label with name \"+3.3VP\""
-			(at 114.3 85.09 0)
-			(effects
-				(font
-					(size 1.27 1.27)
-				)
-				(hide yes)
-			)
-		)
-		(pin "1"
-		)
-		(instances
-			(project "anarchytechnobox"
-				(path "/8c734c41-38ed-40fc-83bd-134786dcfb35/48f260d8-d62f-49a9-8985-05fca65ac6cb"
-					(reference "#PWR057")
-					(unit 1)
-				)
-				(path "/8c734c41-38ed-40fc-83bd-134786dcfb35/f97c65ed-bb3f-4eb8-a2c6-056cc510b5f8"
-					(reference "#PWR065")
-					(unit 1)
-				)
-			)
-		)
-	)
-	(symbol
 		(lib_id "parts:ISO7740")
 		(at 97.79 40.64 0)
@@
 	)
 	(symbol
+		(lib_id "power:+5VP")
+		(at 121.92 40.64 0)
+		(unit 1)
+		(exclude_from_sim no)
+		(in_bom yes)
+		(on_board yes)
+		(dnp no)
+		(fields_autoplaced yes)
+		(property "Reference" "#PWR031"
+			(at 121.92 44.45 0)
+			(effects
+				(font
+					(size 1.27 1.27)
+				)
+				(hide yes)
+			)
+		)
+		(property "Value" "+5VP"
+			(at 121.92 35.56 0)
+			(effects
+				(font
+					(size 1.27 1.27)
+				)
+			)
+		)
+		(property "Footprint" ""
+			(at 121.92 40.64 0)
+			(effects
+				(font
+					(size 1.27 1.27)
+				)
+				(hide yes)
+			)
+		)
+		(property "Datasheet" ""
+			(at 121.92 40.64 0)
+			(effects
+				(font
+					(size 1.27 1.27)
+				)
+				(hide yes)
+			)
+		)
+		(property "Description" "Power symbol creates a global label with name \"+5VP\""
+			(at 121.92 40.64 0)
+			(effects
+				(font
+					(size 1.27 1.27)
+				)
+				(hide yes)
+			)
+		)
+		(pin "1"
+		)
+		(instances
+			(project "anarchytechnobox"
+				(path "/8c734c41-38ed-40fc-83bd-134786dcfb35/48f260d8-d62f-49a9-8985-05fca65ac6cb"
+					(reference "#PWR031")
+					(unit 1)
+				)
+				(path "/8c734c41-38ed-40fc-83bd-134786dcfb35/f97c65ed-bb3f-4eb8-a2c6-056cc510b5f8"
+					(reference "#PWR033")
+					(unit 1)
+				)
+			)
+		)
+	)
+	(symbol
 		(lib_id "Diode:BAT54AW")
 		(at 177.8 93.98 270)
@@
 					(unit 1)
 				)
-			)
-		)
-	)
-	(symbol
-		(lib_id "power:+3.3VP")
-		(at 121.92 40.64 0)
-		(unit 1)
-		(exclude_from_sim no)
-		(in_bom yes)
-		(on_board yes)
-		(dnp no)
-		(fields_autoplaced yes)
-		(property "Reference" "#PWR059"
-			(at 125.73 41.91 0)
-			(effects
-				(font
-					(size 1.27 1.27)
-				)
-				(hide yes)
-			)
-		)
-		(property "Value" "+3.3VP"
-			(at 121.92 35.56 0)
-			(effects
-				(font
-					(size 1.27 1.27)
-				)
-			)
-		)
-		(property "Footprint" ""
-			(at 121.92 40.64 0)
-			(effects
-				(font
-					(size 1.27 1.27)
-				)
-				(hide yes)
-			)
-		)
-		(property "Datasheet" ""
-			(at 121.92 40.64 0)
-			(effects
-				(font
-					(size 1.27 1.27)
-				)
-				(hide yes)
-			)
-		)
-		(property "Description" "Power symbol creates a global label with name \"+3.3VP\""
-			(at 121.92 40.64 0)
-			(effects
-				(font
-					(size 1.27 1.27)
-				)
-				(hide yes)
-			)
-		)
-		(pin "1"
-		)
-		(instances
-			(project "anarchytechnobox"
-				(path "/8c734c41-38ed-40fc-83bd-134786dcfb35/48f260d8-d62f-49a9-8985-05fca65ac6cb"
-					(reference "#PWR059")
-					(unit 1)
-				)
-				(path "/8c734c41-38ed-40fc-83bd-134786dcfb35/f97c65ed-bb3f-4eb8-a2c6-056cc510b5f8"
-					(reference "#PWR067")
-					(unit 1)
-				)

Commit message: Schematic & PCB changes: - Cleaned up unnecessary electrolytic input capacitor flyback - Removed dual diode rectification on 5V, increased output capacitors - Feedback resistors DC/DCs set, enlarged for JLC basic parts - Sweep through schematic to consolidate caps to JLC basic parts (see list schematic front page) - Midi OUTPUT added (please check schematic) - Wiznet W5500 schematic reworked to RJ45 reference schematic: https://docs.wiznet.io/assets/files/w5500_sch_v110_use_mag_-dfff8bbb103d13be4f25cd2b2f8b950d.pdf - Replaced ethernet jack to HR911105A - Crystals chosen for W5500 and RP2350B (according to reference), 15pF load caps. - RS485 driver changed to SP3485EN for 3.3V operation - Replaced RS485 bus connectors with 2x RJ45s for passthrough - Groove connector replaced with JST XH 2mm - Added LCSC part numbers for various components in the schematic
Parts:
- U9: LCSC Part (none) -> C529547
Changed lines of the file:
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@@
 		(at 180.34 135.89)
-	)
-	(bus_entry
-		(at 223.52 44.45)
-		(size 2.54 2.54)
-		(stroke
-			(width 0)
-			(type default)
-		)
 	)
 	(wire
@@
 			(effects
 				(font
+					(size 1.27 1.27)
+				)
+				(hide yes)
+			)
+		)
+		(property "LCSC Part" "C529547"
+			(at 97.79 40.64 0)
+			(effects
+				(font

Commit message: BOM nagelopen, bestelklaar.
Parts:
- D4: LCSC Part (none) -> C2836067
Changed lines of the file:
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@@
+			)
+		)
+		(property "LCSC Part" "C2836067"
+			(at 177.8 93.98 90)
+			(effects
+				(font
+					(size 1.27 1.27)
+				)
+				(hide yes)
 			)
 		)

Commit message: 10k W5500 on RSVD pin
Other:
- note added: "Let op _1 en _2 wisselen hier om"
Changed lines of the file:
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@@
 	(generator_version "9.0")
 	(paper "A4")
+	(text "Let op _1 en _2 wisselen hier om"
+		(exclude_from_sim no)
+		(at 110.236 29.718 0)
+		(effects
+			(font
+				(size 1.27 1.27)
+			)
+		)
+	)
 	(junction
 		(at 92.71 68.58)
